File: PowerExtender_x3.kicad_pcb (KiCad board)
At the start: 2 copper layers, 55.3 x 42.7 mm, 14 parts, among them J1 Conn_01x05, J2 Conn_01x05, J3 Conn_01x05, J4 Conn_01x05, J5 Conn_01x05, J6 Conn_01x05, J7 Conn_01x05, J8 Conn_01x05

Commit message: Label change from "VIN module" to "PnP Power Module"
Other:
- board text added: "PnP Power Module"
- board text removed: "VIN module"
Changed lines of the file:
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@@
 		(layer "Edge.Cuts")
 	)
-	(gr_text "VIN module"
-		(at 91.027144 119.3 0)
+	(gr_text "PnP Power Module"
+		(at 87.538358 119.3 0)
 		(layer "F.SilkS")
 		(effects
@@
 		)
 	)
-	(gr_text "VIN module"
-		(at 118.227144 119.3 0)
+	(gr_text "PnP Power Module"
+		(at 115.078358 119.3 0)
 		(layer "F.SilkS")
 		(effects
@@
 		)
 	)
-	(gr_text "VIN module"
-		(at 101.497357 113.2 180)
+	(gr_text "PnP Power Module"
+		(at 104.812642 113.2 180)
 		(layer "F.SilkS")
 		(effects
@@
 		)
 	)
-	(gr_text "VIN module"
-		(at 129.038357 113.2 180)
+	(gr_text "PnP Power Module"
+		(at 132.352642 113.2 180)
 		(layer "F.SilkS")
 		(effects
