File: panel.kicad_pcb (KiCad board)
At the start: 2 copper layers, 99.4 x 69.3 mm, 40 parts, among them J1 Conn_01x05, J2 Conn_01x05, J3 Conn_01x05, J4 Conn_01x05, J5 Conn_01x05, J6 Conn_01x05, J7 Conn_01x05, J8 Conn_01x05

Commit message: Label change from "VIN module" to "PnP Power Module"
Other:
- board text added: "PnP Power Module"
- board text removed: "VIN module"
